File: hardware/controller.brd (EAGLE design)
At the start: 73.7 x 73.7 mm, 53 parts, among them CON1 LED, CON2 LED, CON3 LED, CON4 LED, IC201 FT232RQ, J301 POWER_JACKPTH, J302 Bulb, U101 STM32F030CC, U201 USB-MICROB, U301 5V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

Commit message: Fix USART1 pins
Connections:
- removed net PA10: U101.31
- removed net PA9: U101.30
- new net PA2: U101.12
- new net PA3: U101.13
- net USART1_RX: now also U101.31; no longer U101.13
- net USART1_TX: now also U101.30; no longer U101.12
Routing:
- net USART1_TX: track 13.6 -> 23.1 mm, vias 0 -> 2
- net USART1_RX: track 10.5 -> 19.6 mm, vias 0 -> 2
Changed lines of the file:
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@@
 </signal>
 <signal name="USART1_TX">
-<contactref element="U101" pad="12"/>
 <contactref element="IC201" pad="2"/>
-<wire x1="22.30445" y1="47.441059375" x2="16.973340625" y2="47.441059375" width="0.2032" layer="1"/>
 <wire x1="16.973340625" y1="47.441059375" x2="14.7828" y2="49.6316" width="0.2032" layer="1"/>
 <wire x1="14.7828" y1="49.6316" x2="14.7828" y2="50.546" width="0.2032" layer="1"/>
@@
 <wire x1="12.172" y1="51.034" x2="12.172" y2="50.306" width="0.2032" layer="1"/>
 <wire x1="14.7828" y1="50.546" x2="13.4874" y2="51.8414" width="0.2032" layer="1"/>
+<contactref element="U101" pad="30"/>
+<wire x1="30.082625" y1="43.19841875" x2="28.01824375" y2="45.2628" width="0.1524" layer="1"/>
+<wire x1="28.01824375" y1="45.2628" x2="27.94" y2="45.2628" width="0.1524" layer="1"/>
+<via x="27.94" y="45.2628" extent="1-16" drill="0.35"/>
+<wire x1="27.94" y1="45.2628" x2="19.1516" y2="45.2628" width="0.1524" layer="16"/>
+<wire x1="19.1516" y1="45.2628" x2="16.973340625" y2="47.441059375" width="0.1524" layer="16"/>
+<via x="16.973340625" y="47.441059375" extent="1-16" drill="0.35"/>
 </signal>
 <signal name="USART1_RX">
-<contactref element="U101" pad="13"/>
 <contactref element="IC201" pad="30"/>
 <wire x1="13.234" y1="48.768" x2="13.222" y2="48.756" width="0.2032" layer="1"/>
-<wire x1="22.30445" y1="45.3197375" x2="17.6214625" y2="45.3197375" width="0.2032" layer="1"/>
 <wire x1="17.6214625" y1="45.3197375" x2="14.1986" y2="48.7426" width="0.2032" layer="1"/>
 <wire x1="14.1986" y1="48.7426" x2="13.2594" y2="48.7426" width="0.2032" layer="1"/>
 <wire x1="13.2594" y1="48.7426" x2="13.234" y2="48.768" width="0.2032" layer="1"/>
+<contactref element="U101" pad="31"/>
+<wire x1="30.436178125" y1="43.551971875" x2="29.7434" y2="44.24475" width="0.1524" layer="1"/>
+<wire x1="29.7434" y1="44.24475" x2="29.7434" y2="44.6024" width="0.1524" layer="1"/>
+<via x="29.7434" y="44.6024" extent="1-16" drill="0.35"/>
+<wire x1="29.7434" y1="44.6024" x2="18.3388" y2="44.6024" width="0.1524" layer="16"/>
+<wire x1="18.3388" y1="44.6024" x2="17.6214625" y2="45.3197375" width="0.1524" layer="16"/>
+<via x="17.6214625" y="45.3197375" extent="1-16" drill="0.35"/>
 </signal>
 <signal name="USART6_TX">
@@
 <signal name="PA11">
 <contactref element="U101" pad="32"/>
-</signal>
-<signal name="PA10">
-<contactref element="U101" pad="31"/>
-</signal>
-<signal name="PA9">
-<contactref element="U101" pad="30"/>
 </signal>
 <signal name="PB15">
@@
 <wire x1="13.6922" y1="3.6966" x2="13.716" y2="3.7204" width="0.2032" layer="1"/>
 </signal>
+<signal name="PA2">
+<contactref element="U101" pad="12"/>
+</signal>
+<signal name="PA3">
+<contactref element="U101" pad="13"/>
+</signal>
 </signals>

Commit message: Hardware updates
Parts:
- removed R203: 10k, lights:R0603
- added C205: 0.1uF, lights:0603-CAP
- added JP101: (no value), lights:1X04
- added JP5: (no value), lights:1X03
- Q1: device lights:ABS25 -> lights:FC1610AN
- moved C106 5.50 mm to (27.8, 59.4)
- moved C107 5.22 mm to (23.7, 59.4)
- moved Q1 2.96 mm to (25.7, 57.9), turned to 0 degrees
Connections:
- net N$9 renamed BULB
- net USART2_RX renamed PA15
- removed net PA13: U101.34
- removed net USART2_TX: U101.37
- new net SWCLK: JP101.2, U101.37
- new net SWDIO: JP101.3, U101.34
- net 3.3V: now also C109.1, JP101.1; no longer R203.1
- net BOOT0: now also JP5.1
- net GND: now also C109.2, C205.1, JP101.4, JP5.3
- net NRST: now also C205.2, JP5.2; no longer R203.2
- net OSC32_IN: now also Q1.2; no longer Q1.4
- net VDDA: no longer C109.1
- net VSSA: no longer C109.2
Routing:
- net SWCLK: track 0.00 -> 30.0 mm, vias 0 -> 2
- net SWDIO: track 0.00 -> 27.6 mm, vias 0 -> 2
- net 3.3V: track 41.7 -> 54.4 mm, vias 8 -> 11
- net BOOT0: track 44.2 -> 51.7 mm, vias 3 -> 2
- net OSC32_IN: track 17.1 -> 10.1 mm
- net OSC32_OUT: track 17.1 -> 10.1 mm
- net GND: track 8.65 -> 14.1 mm, vias 4 -> 8
- net NRST: track 28.9 -> 32.5 mm, vias 2 -> 0
- net VSSA: track 6.96 -> 5.61 mm
- net USART4_RX: track 27.3 -> 28.3 mm
Other:
- board text added: "3.3V"
- board text added: "GND"
- board text added: "SWCLK"
- board text added: "SWDIO"
