File: hardware/controller.sch (EAGLE design)
At the start: 53 parts, among them CON1 LED, CON2 LED, CON3 LED, CON4 LED, IC201 FT232RQ, J301 POWER_JACKPTH, J302 Bulb, U101 STM32F030CC, U201 USB-MICROB, U301 5V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

Commit message: Fix USART1 pins
Connections:
- removed net PA10: U101.PA10
- removed net PA9: U101.PA9
- new net PA2: U101.PA2
- new net PA3: U101.PA3
- net USART1_RX: now also U101.PA10; no longer U101.PA3
- net USART1_TX: now also U101.PA9; no longer U101.PA2
Changed lines of the file:
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@@
 <net name="USART1_TX" class="0">
 <segment>
-<pinref part="U101" gate="G$1" pin="PA2"/>
-<wire x1="109.22" y1="119.38" x2="101.6" y2="119.38" width="0.1524" layer="91"/>
-<label x="101.6" y="119.38" size="1.27" layer="95" rot="R180" xref="yes"/>
+<pinref part="U101" gate="G$1" pin="PA9"/>
+<wire x1="162.56" y1="134.62" x2="154.94" y2="134.62" width="0.1524" layer="91"/>
+<label x="162.56" y="134.62" size="1.27" layer="95" xref="yes"/>
 </segment>
 </net>
 <net name="USART1_RX" class="0">
 <segment>
-<pinref part="U101" gate="G$1" pin="PA3"/>
-<wire x1="109.22" y1="116.84" x2="101.6" y2="116.84" width="0.1524" layer="91"/>
-<label x="101.6" y="116.84" size="1.27" layer="95" rot="R180" xref="yes"/>
+<pinref part="U101" gate="G$1" pin="PA10"/>
+<wire x1="154.94" y1="132.08" x2="162.56" y2="132.08" width="0.1524" layer="91"/>
+<label x="162.56" y="132.08" size="1.27" layer="95" xref="yes"/>
 </segment>
 </net>
@@
 <wire x1="162.56" y1="129.54" x2="154.94" y2="129.54" width="0.1524" layer="91"/>
 <label x="162.56" y="129.54" size="1.27" layer="95" xref="yes"/>
-</segment>
-</net>
-<net name="PA10" class="0">
-<segment>
-<pinref part="U101" gate="G$1" pin="PA10"/>
-<wire x1="154.94" y1="132.08" x2="162.56" y2="132.08" width="0.1524" layer="91"/>
-<label x="162.56" y="132.08" size="1.27" layer="95" xref="yes"/>
-</segment>
-</net>
-<net name="PA9" class="0">
-<segment>
-<pinref part="U101" gate="G$1" pin="PA9"/>
-<wire x1="162.56" y1="134.62" x2="154.94" y2="134.62" width="0.1524" layer="91"/>
-<label x="162.56" y="134.62" size="1.27" layer="95" xref="yes"/>
 </segment>
 </net>
@@
 </segment>
 </net>
+<net name="PA2" class="0">
+<segment>
+<pinref part="U101" gate="G$1" pin="PA2"/>
+<wire x1="109.22" y1="119.38" x2="101.6" y2="119.38" width="0.1524" layer="91"/>
+<label x="101.6" y="119.38" size="1.27" layer="95" rot="R180" xref="yes"/>
+</segment>
+</net>
+<net name="PA3" class="0">
+<segment>
+<pinref part="U101" gate="G$1" pin="PA3"/>
+<wire x1="109.22" y1="116.84" x2="101.6" y2="116.84" width="0.1524" layer="91"/>
+<label x="101.6" y="116.84" size="1.27" layer="95" rot="R180" xref="yes"/>
+</segment>
+</net>

Commit message: Hardware updates
Parts:
- removed R203: 10k, lights:R0603R0603
- added C205: 0.1uF, lights:C0603
- added JP101: (no value), lights:PINHD-1X4
- added JP5: (no value), lights:PINHD-1X3
- Q1: device lights:CRYSTAL -> lights:CRYSTALFC1610AN
Connections:
- net N$9 renamed BULB
- net USART2_RX renamed PA15
- removed net PA13: U101.PA13
- removed net USART2_TX: U101.PA14
- new net SWCLK: JP101.2, U101.PA14
- new net SWDIO: JP101.3, U101.PA13
- net 3.3V: now also C109.1, JP101.1; no longer R203.1
- net BOOT0: now also JP5.1
- net GND: now also C109.2, C205.1, JP101.4, JP5.3
- net NRST: now also C205.2, JP5.2; no longer R203.2
- net VDDA: no longer C109.1
- net VSSA: no longer C109.2
